File: PCB/PCB.kicad_pcb (KiCad board)
At the start: 2 copper layers, 17 parts, among them J1 PWM, J10 3V3, J11 I2C 1.1, J12 I2C 2.1, J13 PWM, J14 I2C 1.2, J15 I2C 2.2, J16 I2C 1.3, J17 I2C 2.3, J2 5V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

Commit message: Add gerber files
Parts:
- J7: value Raspberry_Pi_2_3 -> (none)
Connections:
- J14 pad 2: Net-(J14-Pad2) -> Net-(J11-Pad2)
- J16 pad 2: Net-(J14-Pad2) -> Net-(J11-Pad2)
Routing:
- net Net-(J11-Pad2): track 0.00 -> 154.2 mm
- net Net-(J4-Pad1): track 0.00 -> 134.7 mm, vias 0 -> 1
- net Net-(J1-Pad2): track 0.00 -> 111.6 mm, vias 0 -> 1
- net Net-(J2-Pad1): track 0.00 -> 105.1 mm
- net Net-(J10-Pad1): track 0.00 -> 77.4 mm
- net Net-(J11-Pad1): track 0.00 -> 60.9 mm, vias 0 -> 1
- net Net-(J12-Pad2): track 0.00 -> 44.3 mm
- net Net-(J12-Pad1): track 0.00 -> 38.9 mm
- net Net-(J1-Pad1): track 0.00 -> 22.3 mm, vias 0 -> 1
- net Net-(J13-Pad2): track 0.00 -> 19.1 mm, vias 0 -> 1
- net Net-(J13-Pad1): track 0.00 -> 12.2 mm
- added copper zone on B.Cu, net (none)
- added copper zone on F.Cu, net Net-(J4-Pad1)
Other:
- board outline added: 50 x 68 mm
- board text added: "1072 Raspi Breakout"
